File: pressure.kicad_sch (KiCad schematic)
At the start: 43 parts, among them IC5 ADS131M04IRUKR, J4 1053131104, J5 1053131104, J6 1053131104

Commit message: Updated TVS diode
Parts:
- added IC3: ADS131M03IRUKR, QFN40P300X300X80-21N-D, symbol ADS131M03IRUKR:ADS131M03IRUKR
Changed lines of the file:
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@@
+	)
+	(symbol
+		(lib_id "ADS131M03IRUKR:ADS131M03IRUKR")
+		(at 29.21 140.97 0)
+		(unit 1)
+		(exclude_from_sim no)
+		(in_bom yes)
+		(on_board yes)
+		(dnp no)
+		(fields_autoplaced yes)
+		(property "Reference" "IC3"
+			(at 64.77 134.5498 0)
+			(effects
+				(font
+					(size 1.27 1.27)
+				)
+			)
+		)
+		(property "Value" "ADS131M03IRUKR"
+			(at 64.77 137.0898 0)
+			(effects
+				(font
+					(size 1.27 1.27)
+				)
+			)
+		)
+		(property "Footprint" "QFN40P300X300X80-21N-D"
+			(at 55.88 225.73 0)
+			(effects
+				(font
+					(size 1.27 1.27)
+				)
+				(justify left top)
+				(hide yes)
+			)
+		)
+		(property "Datasheet" "https://www.ti.com/general/docs/suppproductinfo.tsp?distId=10&gotoUrl=http%3A%2F%2Fwww.ti.com%2Flit%2Fgpn%2Fads131m03"
+			(at 55.88 325.73 0)
+			(effects
+				(font
+					(size 1.27 1.27)
+				)
+				(justify left top)
+				(hide yes)
+			)
+		)
+		(property "Description" "Encoders, Decoders, Multiplexers & Demultiplexers 24-bit, 32-kSPS, 3-channel, simultaneous-sampling, delta-sigma ADC 20-WQFN -40 to 125"
+			(at 29.21 140.97 0)
+			(effects
+				(font
+					(size 1.27 1.27)
+				)
+				(hide yes)
+			)
+		)
+		(property "Height" "0.8"
+			(at 55.88 525.73 0)
+			(effects
+				(font
+					(size 1.27 1.27)
+				)
+				(justify left top)
+				(hide yes)
+			)
+		)
+		(property "Mouser Part Number" "595-ADS131M03IRUKR"
+			(at 55.88 625.73 0)
+			(effects
+				(font
+					(size 1.27 1.27)
+				)
+				(justify left top)
+				(hide yes)
+			)
+		)
+		(property "Mouser Price/Stock" "https://www.mouser.co.uk/ProductDetail/Texas-Instruments/ADS131M03IRUKR?qs=stqOd1AaK7%252Bm3QT30xDCgA%3D%3D"
+			(at 55.88 725.73 0)
+			(effects
+				(font
+					(size 1.27 1.27)
+				)
+				(justify left top)
+				(hide yes)
+			)
+		)
+		(property "Manufacturer_Name" "Texas Instruments"
+			(at 55.88 825.73 0)
+			(effects
+				(font
+					(size 1.27 1.27)
+				)
+				(justify left top)
+				(hide yes)
+			)
+		)
+		(property "Manufacturer_Part_Number" "ADS131M03IRUKR"
+			(at 55.88 925.73 0)
+			(effects
+				(font
+					(size 1.27 1.27)
+				)
+				(justify left top)
+				(hide yes)
+			)
+		)
+		(pin "1"
+		)
+		(pin "6"
+		)
+		(pin "18"
+		)
+		(pin "9"
+		)
+		(pin "14"
+		)
+		(pin "13"
+		)
+		(pin "2"
+		)
+		(pin "17"
+		)
+		(pin "15"
+		)
+		(pin "3"
+		)
+		(pin "4"
+		)
+		(pin "16"
+		)
+		(pin "11"
+		)
+		(pin "21"
+		)
+		(pin "5"
+		)
+		(pin "7"
+		)
+		(pin "20"
+		)
+		(pin "19"
+		)
+		(pin "8"
+		)
+		(pin "10"
+		)
+		(pin "12"
+		)
+		(instances
+			(project ""
+				(path "/7db990e4-92e1-4f99-b4d2-435bbec1ba83/3af81d2a-0ad1-4f51-8454-076646dec8d9"
+					(reference "IC3")
+					(unit 1)
+				)
+			)
+		)
 	)
 	(symbol
