File: servo.kicad_sch (KiCad schematic)
At the start: 3 parts, among them J3 ServoConnector1

Commit message: Updated TVS diode
Parts:
- removed D3: ~, Package_TO_SOT_SMD:SOT-353_SC-70-5, symbol iclr:CPDV5-3V3UP
- added D4: SET23A03L02, SOT95P230X109-3N, symbol SET23A03L02:SET23A03L02
Connections:
- net GND: now also D4.3 (COM_A)
- net ServoPWM: now also D4.1 (K1)
Changed lines of the file:
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@@
+	(wire
+		(pts
+			(xy 115.57 71.12) (xy 118.11 71.12)
+		)
+		(stroke
+			(width 0)
+			(type default)
+		)
+	)
 	(wire
 		(pts
@@
 	(hierarchical_label "ServoPWM"
 		(shape input)
-		(at 154.94 67.31 90)
+		(at 115.57 71.12 180)
 		(effects
 			(font
 				(size 1.27 1.27)
 			)
-			(justify left)
+			(justify right)
 		)
 	)
@@
 			)
 			(justify left)
+		)
+	)
+	(symbol
+		(lib_id "SET23A03L02:SET23A03L02")
+		(at 118.11 71.12 0)
+		(unit 1)
+		(exclude_from_sim no)
+		(in_bom yes)
+		(on_board yes)
+		(dnp no)
+		(fields_autoplaced yes)
+		(property "Reference" "D4"
+			(at 132.08 63.5 0)
+			(effects
+				(font
+					(size 1.27 1.27)
+				)
+			)
+		)
+		(property "Value" "SET23A03L02"
+			(at 132.08 66.04 0)
+			(effects
+				(font
+					(size 1.27 1.27)
+				)
+			)
+		)
+		(property "Footprint" "SOT95P230X109-3N"
+			(at 142.24 166.04 0)
+			(effects
+				(font
+					(size 1.27 1.27)
+				)
+				(justify left top)
+				(hide yes)
+			)
+		)
+		(property "Datasheet" ""
+			(at 142.24 266.04 0)
+			(effects
+				(font
+					(size 1.27 1.27)
+				)
+				(justify left top)
+				(hide yes)
+			)
+		)
+		(property "Description" "ESD Protection Diodes / TVS Diodes TVS ESD SOIC-08 3.3V 76.8V"
+			(at 118.11 71.12 0)
+			(effects
+				(font
+					(size 1.27 1.27)
+				)
+				(hide yes)
+			)
+		)
+		(property "Height" "1.09"
+			(at 142.24 466.04 0)
+			(effects
+				(font
+					(size 1.27 1.27)
+				)
+				(justify left top)
+				(hide yes)
+			)
+		)
+		(property "Mouser Part Number" "603-SET23A03L02"
+			(at 142.24 566.04 0)
+			(effects
+				(font
+					(size 1.27 1.27)
+				)
+				(justify left top)
+				(hide yes)
+			)
+		)
+		(property "Mouser Price/Stock" "https://www.mouser.co.uk/ProductDetail/YAGEO/SET23A03L02?qs=DRkmTr78QASD5DRaK8Y6sQ%3D%3D"
+			(at 142.24 666.04 0)
+			(effects
+				(font
+					(size 1.27 1.27)
+				)
+				(justify left top)
+				(hide yes)
+			)
+		)
+		(property "Manufacturer_Name" "YAGEO"
+			(at 142.24 766.04 0)
+			(effects
+				(font
+					(size 1.27 1.27)
+				)
+				(justify left top)
+				(hide yes)
+			)
+		)
+		(property "Manufacturer_Part_Number" "SET23A03L02"
+			(at 142.24 866.04 0)
+			(effects
+				(font
+					(size 1.27 1.27)
+				)
+				(justify left top)
+				(hide yes)
+			)
+		)
+		(pin "1"
+		)
+		(pin "3"
+		)
+		(pin "2"
+		)
+		(instances
+			(project ""
+				(path "/7db990e4-92e1-4f99-b4d2-435bbec1ba83/55ab0687-c91f-4545-a2ea-e93947dc2af8"
+					(reference "D4")
+					(unit 1)
+				)
+			)
 		)
 	)
@@
 	(symbol
 		(lib_id "power:GND")
-		(at 154.94 80.01 0)
+		(at 146.05 71.12 0)
 		(unit 1)
 		(exclude_from_sim no)
@@
 		(dnp no)
 		(property "Reference" "#PWR046"
-			(at 154.94 86.36 0)
+			(at 146.05 77.47 0)
 			(effects
 				(font
@@
 		)
 		(property "Value" "GND"
-			(at 155.067 83.2612 90)
+			(at 146.177 74.3712 90)
 			(effects
 				(font
@@
 		)
 		(property "Footprint" ""
-			(at 154.94 80.01 0)
+			(at 146.05 71.12 0)
 			(effects
 				(font
@@
 		)
 		(property "Datasheet" ""
-			(at 154.94 80.01 0)
+			(at 146.05 71.12 0)
 			(effects
 				(font
@@
 		)
 		(property "Description" ""
-			(at 154.94 80.01 0)
+			(at 146.05 71.12 0)
 			(effects
 				(font
@@
 					(unit 1)
 				)
-			)
-		)
-	)
-	(symbol
-		(lib_id "iclr:CPDV5-3V3UP")
-		(at 154.94 58.42 0)
-		(unit 1)
-		(exclude_from_sim no)
-		(in_bom yes)
-		(on_board yes)
-		(dnp no)
-		(property "Reference" "D3"
-			(at 152.908 73.66 0)
-			(effects
-				(font
-					(size 1.27 1.27)
-				)
-				(justify right)
-			)
-		)
-		(property "Value" "~"
-			(at 152.4 74.93 0)
-			(effects
-				(font
-					(size 1.27 1.27)
-				)
-				(justify right)
-			)
-		)
-		(property "Footprint" "Package_TO_SOT_SMD:SOT-353_SC-70-5"
-			(at 154.94 68.58 0)
-			(effects
-				(font
-					(size 1.27 1.27)
-				)
-				(hide yes)
-			)
-		)
-		(property "Datasheet" "https://www.mouser.co.uk/datasheet/2/80/CPDV5_3V3UP_HF_RevB181493-2505215.pdf"
-			(at 154.94 68.58 0)
-			(effects
-				(font
-					(size 1.27 1.27)
-				)
-				(hide yes)
-			)
-		)
-		(property "Description" "2 channel double backed zener TVS diode"
-			(at 154.94 68.58 0)
-			(effects
-				(font
-					(size 1.27 1.27)
-				)
-				(hide yes)
-			)
-		)
-		(pin "4"
-		)
-		(pin "2"
-		)
-		(pin "5"
-		)
-		(pin "3"
-		)
-		(pin "1"
-		)
-		(pin "2"
-		)
-		(instances
-			(project "RicardoTemplate"
-				(path "/7db990e4-92e1-4f99-b4d2-435bbec1ba83/55ab0687-c91f-4545-a2ea-e93947dc2af8"
-					(reference "D3")
-					(unit 1)
-				)
